Commit message: feat: ABA working

File: resource/kinova/robot_no_fixed.urdf (robot description, URDF)
Before this commit: robot kinova, 4 links, 3 joints
Links:
- added link kinova_link_3, mass 0.6763; visual mesh filename=../meshes/forearm.dae; visual mesh filename=../meshes/ring_big.STL
Joints:
- added joint kinova_joint_3: type revolute, parent kinova_link_2, child kinova_link_3, origin xyz=0 -0.410 0 rpy=0 3.14159265359 0, axis 0 0 1, limit lower=-62.8318530718 upper=62.8318530718 effort=30.5 velocity=15
