Commit message: feat: kinematics work

File: resource/chain/robot.urdf (robot description, URDF)
Before this commit: robot 2DrobotArm, 5 links, 4 joints
Links:
- link link1: geometry visual sphere radius=0.1
- link link2: geometry visual sphere radius=0.1
- link link3: geometry visual sphere radius=0.1
- link link4: geometry visual sphere radius=0.1
